Commit message: finish velocity commander

File: urdf/stretch_pruned.urdf (robot description, URDF)
Before this commit: robot stretch, 14 links, 13 joints
Links:
- removed link link_head_teleop_camera
- removed link link_head_teleop_mount
- added link link_base_revolution, mass 1.0
- link base_link: geometry 
- link link_arm_l0: geometry 
- link link_arm_l1: geometry 
- link link_arm_l2: geometry 
- link link_arm_l3: geometry 
- link link_arm_l4: geometry 
- link link_gripper: geometry 
- link link_lift: geometry 
- link link_mast: geometry 
- link link_wrist_yaw: geometry 
Joints:
- removed joint joint_head_teleop_camera
- removed joint joint_head_teleop_mount
- added joint joint_base_revolution: type revolute, parent link_base_translation, child link_base_revolution, origin xyz=0.0 0.0 0.0 rpy=0.0 -0.0 0.0, axis 0. 0. 1., limit lower=-3.0 upper=3.0 effort=100.0 velocity=1.0
- joint joint_base_translation: limit lower=-1.0 upper=1.0 effort=100.0 velocity=1.0 -> lower=-3.0 upper=3.0 effort=100.0 velocity=1.0
- joint joint_mast: parent link_base_translation -> link_base_revolution
