Commit message: calibrate stretch and add some readme

File: da_core/urdf/stretch_pruned.urdf (robot description, URDF)
Before this commit: robot stretch, 13 links, 12 joints
Joints:
- joint joint_arm_l4: origin xyz=-0.2547 0.0 0.0 rpy=1.5708 2.4721e-15 -1.5708 -> xyz=-0.251582752247285 -0.006070296440143875 -0.005254623139652845 rpy=1.5664162057374356 0.059620207701978734 -1.5661623604639134
- joint joint_mast: origin xyz=-0.067 0.135 0.0284 rpy=1.5708 0.0 4.8006e-17 -> xyz=-0.07009055762807098 0.13159786057784964 0.028302116135615125 rpy=1.5648678330247587 0.013954114010035212 -0.02346559894719587
